Commit message: Solved some bugs

File: SinglePendulum_cpp/single_pendulum_description/urdf/single_pendulum.urdf (robot description, URDF)
Before this commit: robot 2dof_planar, 2 links, 1 joints
Links:
- link link1: mass 0.14 -> 0.26703

Commit message: Bug fixes.

File: SinglePendulum_cpp/single_pendulum_description/urdf/single_pendulum.urdf (robot description, URDF)
Before this commit: robot 2dof_planar, 2 links, 1 joints
Links:
- link base_link: mass 0.10159 -> None
- link link1: mass 0.26703 -> 0.14
Joints:
- joint joint1: origin xyz=0.0060872 0 0.035 rpy=0 0 0 -> xyz=0 0 0 rpy=0 0 0
